Commit message: Refactor: Reorganize URDF files, added inertia and collision boxes

File: src/my_robot_description/urdf/common_properties.xacro (robot description, xacro)
@@ -1,27 +1,45 @@
 <?xml version="1.0"?>
 <robot xmlns:xacro="http://www.ros.org/wiki/xacro">
-    <material name="blue">
-        <color rgba="0 0 0.5 1" />
-    </material>
-    <material name="grey">
-        <color rgba="0.5 0.5 0.5 1" />
-    </material>
-    <material name="red">
-        <color rgba="0.8 0 0 1"/>
-    </material>
-    <material name="green">
-        <color rgba="0 0.8 0 1"/>
-    </material>
-    <material name="yellow">
-        <color rgba="0.8 0.8 0 1"/>
-    </material>
-  <!-- Visual Properties -->
-  <xacro:property name="body_color_rgba" value="0.3 0.3 0.8 1.0"/>
-  <!-- Color definitions -->
-  <xacro:property name="color_green" value="0.2 0.8 0.2 1.0"/>
-  <xacro:property name="color_cyan" value="0.0 0.8 0.8 1.0"/>
-  <xacro:property name="color_red" value="0.8 0.2 0.2 1.0"/>
-  <xacro:property name="color_orange" value="1.0 0.5 0.0 1.0"/>
-  <xacro:property name="color_yellow" value="1.0 1.0 0.0 1.0"/>
-  <xacro:property name="color_violet" value="0.5 0.0 0.5 1.0"/>
+    <!-- Visual Properties -->
+    <xacro:property name="body_color_rgba" value="0.3 0.3 0.8 1.0"/>
+    <!-- Color definitions -->
+    <xacro:property name="color_green" value="0.2 0.8 0.2 1.0"/>
+    <xacro:property name="color_cyan" value="0.0 0.8 0.8 1.0"/>
+    <xacro:property name="color_red" value="0.8 0.2 0.2 1.0"/>
+    <xacro:property name="color_orange" value="1.0 0.5 0.0 1.0"/>
+    <xacro:property name="color_yellow" value="1.0 1.0 0.0 1.0"/>
+    <xacro:property name="color_violet" value="0.5 0.0 0.5 1.0"/>
+    <!-- inertia definitions -->
+    <xacro:property name="base_link_mass" value="0.5"/>
+    <xacro:property name="leg_segment_mass" value="0.1167"/>
+    <xacro:macro name="box_inertia" params="m x y z">
+        <inertial>
+        <origin xyz="0 0 0" rpy="0 0 0"/>
+        <mass value="${m}"/>
+        <inertia  ixx="${m/12 * (y*y + z*z)}" ixy="0" ixz="0"
+                    iyy="${m/12 * (x*x + z*z)}" iyz="0"
+                    izz="${m/12 * (x*x + y*y)}"/>
+        </inertial>
+    </xacro:macro>
+    <xacro:macro name="base_link_inertial">
+        <xacro:box_inertia m="${base_link_mass}"
+                        x="${body_length}"
+                        y="${body_width}"
+                        z="${body_height}"/>
+    </xacro:macro>
+    <xacro:macro name="leg_segment_inertial" params="x y z">
+        <xacro:box_inertia m="${leg_segment_mass}"
+                        x="${x}"
+                        y="${y}"
+                        z="${z}"/>
+    </xacro:macro>
+    <!-- collision definitions -->
+    <xacro:macro name="box_collision" params="x y z">
+      <collision>
+        <origin xyz="0 0 0" rpy="0 0 0"/>
+        <geometry>
+          <box size="${x} ${y} ${z}"/>
+        </geometry>
+      </collision>
+    </xacro:macro>
 </robot>

File: src/my_robot_description/urdf/mobile_base.xacro (robot description, xacro)
@@ -6,36 +6,6 @@
 -->
 <robot name="hexapod" xmlns:xacro="http://ros.org/wiki/xacro">
-  <!-- Body Parameters -->
-  <xacro:property name="body_start_pos" value="0.1"/>  <!-- desired distance from ground to bottom of body -->
-  <xacro:property name="body_length" value="0.175"/>
-  <xacro:property name="body_width" value="0.130"/>
-  <xacro:property name="body_width_middle" value="0.170"/>
-  <xacro:property name="body_height" value="0.043"/>
-  <!-- Leg Segment Parameters -->
-  <!-- Coxa (Hip) -->
-  <xacro:property name="coxa_length" value="0.0436"/>
-  <xacro:property name="coxa_width"  value="0.0254"/>
-  <xacro:property name="coxa_height" value="0.0582"/>
-  <!-- Femur (Thigh) -->
-  <xacro:property name="femur_length" value="0.07994"/>
-  <xacro:property name="femur_width"  value="0.059"/>
-  <xacro:property name="femur_height" value="0.02"/>
-  <!-- Tibia (Shin) -->
-  <xacro:property name="tibia_length" value="0.1787"/>
-  <xacro:property name="tibia_width"  value="0.012"/>
-  <xacro:property name="tibia_height" value="0.012"/>
-  <!-- Joint Limits -->
-  <xacro:property name="coxa_joint_limit" value="1.57"/>
-  <xacro:property name="femur_joint_limit" value="1.57"/> <!-- 90 degrees -->
-  <xacro:property name="tibia_joint_limit" value="1.5"/>  <!-- ~86 degrees -->
-  <!-- Computed Properties -->
-  <xacro:property name="half_body_height" value="${body_height/2}"/>
-  <xacro:property name="half_body_width"  value="${body_width/2}"/>
-  <xacro:property name="half_coxa_width"  value="${coxa_width/2}"/>
   <!-- base_footprint empty frame at world z=0 -->
   <link name="base_footprint"/>
-  <!-- Leg mounting position -->
-  <xacro:property name="leg_mount_z" value="${body_height/2}"/>  <!-- z offset for leg mounting points -->
-  <!-- base_link robot body center -->
   <link name="base_link">
     <visual>
@@ -48,6 +18,20 @@
       </material>
     </visual>
+    <inertial>
+      <mass value="${base_link_mass}"/>
+      <origin xyz="0 0 ${body_height/2}" rpy="0 0 0"/>
+      <inertia  ixx="${base_link_mass/12 * (body_width*body_width + body_height*body_height)}"
+                ixy="0" ixz="0"
+                iyy="${base_link_mass/12 * (body_length*body_length + body_height*body_height)}"
+                iyz="0"
+                izz="${base_link_mass/12 * (body_length*body_length + body_width*body_width)}"/>
+    </inertial>
+    <collision>
+      <geometry>
+        <box size="${body_length} ${body_width} ${body_height}"/>
+      </geometry>
+      <origin xyz="0 0 ${body_height/2}" rpy="0 0 0"/>
+    </collision>
   </link>
-  <!-- Joint connecting base_footprint to base_link -->
   <joint name="base_footprint_to_base_link" type="fixed">
     <parent link="base_footprint"/>
@@ -67,5 +51,4 @@
   -->
   <xacro:macro name="leg" params="prefix parent x y z roll pitch yaw color_rgba">
-    <!-- Coxa (hip) link and joint -->
     <link name="${prefix}_coxa_link">
       <visual>
@@ -76,4 +59,19 @@
         <material name="${prefix}_material_coxa"><color rgba="${color_rgba}"/></material>
       </visual>
+      <inertial>
+        <mass value="${leg_segment_mass}"/>
+        <origin xyz="${coxa_length/2} 0 0" rpy="0 0 0"/>
+        <inertia  ixx="${leg_segment_mass/12 * (coxa_width*coxa_width + coxa_height*coxa_height)}"
+                  ixy="0" ixz="0"
+                  iyy="${leg_segment_mass/12 * (coxa_length*coxa_length + coxa_height*coxa_height)}"
+                  iyz="0"
+                  izz="${leg_segment_mass/12 * (coxa_length*coxa_length + coxa_width*coxa_width)}"/>
+      </inertial>
+      <collision>
+        <origin xyz="${coxa_length/2} 0 0" rpy="0 0 0"/>
+        <geometry>
+          <box size="${coxa_length} ${coxa_width} ${coxa_height}"/>
+        </geometry>
+      </collision>
     </link>
     <joint name="${prefix}_base_to_coxa_joint" type="revolute">
@@ -84,5 +82,4 @@
       <limit lower="${-coxa_joint_limit}" upper="${coxa_joint_limit}" effort="5.0" velocity="2.0"/>
     </joint>
-    <!-- Femur (thigh) link and joint -->
     <link name="${prefix}_femur_link">
       <visual>
@@ -93,4 +90,19 @@
         <material name="${prefix}_material_femur"><color rgba="${color_rgba}"/></material>
       </visual>
+      <inertial>
+        <mass value="${leg_segment_mass}"/>
+        <origin xyz="${femur_length/2} 0 0" rpy="0 0 0"/>
+        <inertia  ixx="${leg_segment_mass/12 * (femur_width*femur_width + femur_height*femur_height)}"
+                  ixy="0" ixz="0"
+                  iyy="${leg_segment_mass/12 * (femur_length*femur_length + femur_height*femur_height)}"
+                  iyz="0"
+                  izz="${leg_segment_mass/12 * (femur_length*femur_length + femur_width*femur_width)}"/>
+      </inertial>
+      <collision>
+        <origin xyz="${femur_length/2} 0 0" rpy="0 0 0"/>
+        <geometry>
+          <box size="${femur_length} ${femur_width} ${femur_height}"/>
+        </geometry>
+      </collision>
     </link>
     <joint name="${prefix}_coxa_to_femur_joint" type="revolute">
@@ -101,5 +113,4 @@
       <limit lower="${-femur_joint_limit}" upper="${femur_joint_limit}" effort="5.0" velocity="2.0"/>
     </joint>
-    <!-- Tibia (shin) link and joint -->
     <link name="${prefix}_tibia_link">
       <visual>
@@ -110,4 +121,19 @@
         <material name="${prefix}_material_tibia"><color rgba="${color_rgba}"/></material>
       </visual>
+      <inertial>
+        <mass value="${leg_segment_mass}"/>
+        <origin xyz="${tibia_length/2} 0 0" rpy="0 0 0"/>
+        <inertia  ixx="${leg_segment_mass/12 * (tibia_width*tibia_width + tibia_height*tibia_height)}"
+                  ixy="0" ixz="0"
+                  iyy="${leg_segment_mass/12 * (tibia_length*tibia_length + tibia_height*tibia_height)}"
+                  iyz="0"
+                  izz="${leg_segment_mass/12 * (tibia_length*tibia_length + tibia_width*tibia_width)}"/>
+      </inertial>
+      <collision>
+        <origin xyz="${tibia_length/2} 0 0" rpy="0 0 0"/>
+        <geometry>
+          <box size="${tibia_length} ${tibia_width} ${tibia_height}"/>
+        </geometry>
+      </collision>
     </link>
     <joint name="${prefix}_femur_to_tibia_joint" type="revolute">
@@ -118,5 +144,5 @@
       <limit lower="${-tibia_joint_limit}" upper="${tibia_joint_limit}" effort="5.0" velocity="2.0"/>
     </joint>
-  </xacro:macro>
+</xacro:macro>
   <!-- Front legs (45 degrees orientation) -->
   <xacro:leg prefix="leg_fr" parent="base_link"

File: src/my_robot_description/urdf/my_robot.urdf.xacro (robot description, xacro)
@@ -1,5 +1,9 @@
 <?xml version="1.0"?>
 <robot name="my_robot" xmlns:xacro="http://www.ros.org/wiki/xacro">
+    <!-- Physical properties of the hexapod -->
+    <xacro:include filename="my_robot_physical_properties.xacro" />
+    <!-- Common properties (colors, inertia macros, etc.) -->
     <xacro:include filename="common_properties.xacro" />
+    <!-- Robot structure -->
     <xacro:include filename="mobile_base.xacro" />
 </robot>

Commit message: Add Gazebo support and update URDF files. Add my_robot_bringup package for Gazebo launch files. Some issues after spawning the robot at gazebo after few minutes, if change the robot position, it does not crash.

File: src/my_robot_description/urdf/common_properties.xacro (robot description, xacro)
@@ -13,7 +13,7 @@
     <xacro:property name="base_link_mass" value="0.5"/>
     <xacro:property name="leg_segment_mass" value="0.1167"/>
-    <xacro:macro name="box_inertia" params="m x y z">
+    <xacro:macro name="box_inertia" params="m x y z origin_x:=0 origin_y:=0 origin_z:=0">
         <inertial>
-        <origin xyz="0 0 0" rpy="0 0 0"/>
+        <origin xyz="${origin_x} ${origin_y} ${origin_z}" rpy="0 0 0"/>
         <mass value="${m}"/>
         <inertia  ixx="${m/12 * (y*y + z*z)}" ixy="0" ixz="0"
@@ -26,5 +26,6 @@
                         x="${body_length}"
                         y="${body_width}"
-                        z="${body_height}"/>
+                        z="${body_height}"
+                        origin_x="0" origin_y="0" origin_z="${body_height/2}"/>
     </xacro:macro>
     <xacro:macro name="leg_segment_inertial" params="x y z">
@@ -32,5 +33,6 @@
                         x="${x}"
                         y="${y}"
-                        z="${z}"/>
+                        z="${z}"
+                        origin_x="${x/2}" origin_y="0" origin_z="0"/>
     </xacro:macro>
     <!-- collision definitions -->

File: src/my_robot_description/urdf/mobile_base.xacro (robot description, xacro)
@@ -18,13 +18,5 @@
       </material>
     </visual>
-    <inertial>
-      <mass value="${base_link_mass}"/>
-      <origin xyz="0 0 ${body_height/2}" rpy="0 0 0"/>
-      <inertia  ixx="${base_link_mass/12 * (body_width*body_width + body_height*body_height)}"
-                ixy="0" ixz="0"
-                iyy="${base_link_mass/12 * (body_length*body_length + body_height*body_height)}"
-                iyz="0"
-                izz="${base_link_mass/12 * (body_length*body_length + body_width*body_width)}"/>
-    </inertial>
+    <xacro:base_link_inertial/>
     <collision>
       <geometry>
@@ -59,13 +51,5 @@
         <material name="${prefix}_material_coxa"><color rgba="${color_rgba}"/></material>
       </visual>
-      <inertial>
-        <mass value="${leg_segment_mass}"/>
-        <origin xyz="${coxa_length/2} 0 0" rpy="0 0 0"/>
-        <inertia  ixx="${leg_segment_mass/12 * (coxa_width*coxa_width + coxa_height*coxa_height)}"
-                  ixy="0" ixz="0"
-                  iyy="${leg_segment_mass/12 * (coxa_length*coxa_length + coxa_height*coxa_height)}"
-                  iyz="0"
-                  izz="${leg_segment_mass/12 * (coxa_length*coxa_length + coxa_width*coxa_width)}"/>
-      </inertial>
+      <xacro:leg_segment_inertial x="${coxa_length}" y="${coxa_width}" z="${coxa_height}"/>
       <collision>
         <origin xyz="${coxa_length/2} 0 0" rpy="0 0 0"/>
@@ -90,13 +74,5 @@
         <material name="${prefix}_material_femur"><color rgba="${color_rgba}"/></material>
       </visual>
-      <inertial>
-        <mass value="${leg_segment_mass}"/>
-        <origin xyz="${femur_length/2} 0 0" rpy="0 0 0"/>
-        <inertia  ixx="${leg_segment_mass/12 * (femur_width*femur_width + femur_height*femur_height)}"
-                  ixy="0" ixz="0"
-                  iyy="${leg_segment_mass/12 * (femur_length*femur_length + femur_height*femur_height)}"
-                  iyz="0"
-                  izz="${leg_segment_mass/12 * (femur_length*femur_length + femur_width*femur_width)}"/>
-      </inertial>
+      <xacro:leg_segment_inertial x="${femur_length}" y="${femur_width}" z="${femur_height}"/>
       <collision>
         <origin xyz="${femur_length/2} 0 0" rpy="0 0 0"/>
@@ -121,13 +97,5 @@
         <material name="${prefix}_material_tibia"><color rgba="${color_rgba}"/></material>
       </visual>
-      <inertial>
-        <mass value="${leg_segment_mass}"/>
-        <origin xyz="${tibia_length/2} 0 0" rpy="0 0 0"/>
-        <inertia  ixx="${leg_segment_mass/12 * (tibia_width*tibia_width + tibia_height*tibia_height)}"
-                  ixy="0" ixz="0"
-                  iyy="${leg_segment_mass/12 * (tibia_length*tibia_length + tibia_height*tibia_height)}"
-                  iyz="0"
-                  izz="${leg_segment_mass/12 * (tibia_length*tibia_length + tibia_width*tibia_width)}"/>
-      </inertial>
+      <xacro:leg_segment_inertial x="${tibia_length}" y="${tibia_width}" z="${tibia_height}"/>
       <collision>
         <origin xyz="${tibia_length/2} 0 0" rpy="0 0 0"/>

File: src/my_robot_description/urdf/my_robot.urdf.xacro (robot description, xacro)
@@ -7,3 +7,5 @@
     <!-- Robot structure -->
     <xacro:include filename="mobile_base.xacro" />
+    <!-- Gazebo properties, uncomment the line if dont want to use gazebo -->
+    <!-- <xacro:include filename="mobile_base_gazebo.xacro" /> -->
 </robot>
