Commit message: phase 2 stage b finished

File: src/hexapod_description/urdf/inertials.xacro (robot description, xacro)
@@ -15,3 +15,14 @@
     </inertial>
   </xacro:macro>
+  <xacro:macro name="sphere_inertia" params="mass radius">
+    <inertial>
+      <mass value="${mass}"/>
+      <inertia
+        ixx="${max((2.0/5.0)*mass*radius*radius, inertia_min)}"
+        ixy="0.0" ixz="0.0"
+        iyy="${max((2.0/5.0)*mass*radius*radius, inertia_min)}"
+        iyz="0.0"
+        izz="${max((2.0/5.0)*mass*radius*radius, inertia_min)}"/>
+    </inertial>
+  </xacro:macro>
 </robot>

File: src/hexapod_description/urdf/leg.xacro (robot description, xacro)
@@ -81,5 +81,24 @@
                          x="${tibia_length}" y="${tibia_width}" z="${tibia_height}"/>
     </link>
-    <!-- Foot-Link wird in Stufe B ergaenzt -->
+    <!-- ===== Foot (Kugel am Tibia-Ende, Punktkontakt + TCP-Frame) ===== -->
+    <joint name="leg_${id}_foot_joint" type="fixed">
+      <parent link="leg_${id}_tibia_link"/>
+      <child  link="leg_${id}_foot_link"/>
+      <origin xyz="${tibia_length} 0 0" rpy="0 0 0"/>
+    </joint>
+    <link name="leg_${id}_foot_link">
+      <visual>
+        <geometry>
+          <sphere radius="${foot_radius}"/>
+        </geometry>
+        <material name="black"/>
+      </visual>
+      <collision>
+        <geometry>
+          <sphere radius="${foot_radius}"/>
+        </geometry>
+      </collision>
+      <xacro:sphere_inertia mass="${foot_mass}" radius="${foot_radius}"/>
+    </link>
   </xacro:macro>
 </robot>
