Commit message: improve connection of the legs to the body

File: src/hexapod_description/urdf/hexapod_physical_properties.xacro (robot description, xacro)
@@ -30,5 +30,9 @@
   <xacro:property name="joint_effort"   value="5.0"/>  <!-- effort/velocity: vom Servo-DB -->
   <xacro:property name="joint_velocity" value="2.0"/>
-  <!-- Mountpunkt-Hoehe der Beine relativ zu base_link -->
-  <xacro:property name="leg_mount_z" value="${body_height/2}"/>
+  <!-- Mountpunkt-Hoehe der Beine relativ zu base_link.
+       Joint-Achse sitzt in der Chassis-Z-Mitte, sodass die Coxa-Box
+       (Z-symmetrisch um den Joint) zentriert um die Chassis-Mittelebene
+       liegt und gleichmaessig oben/unten ueberragt
+       (coxa_height > body_height). Siehe 00_conventions.md §11.3. -->
+  <xacro:property name="leg_mount_z" value="0"/>
 </robot>

Commit message: phase 10 stage f, changed tibia lengh

File: src/hexapod_description/urdf/hexapod_physical_properties.xacro (robot description, xacro)
@@ -14,5 +14,5 @@
   <xacro:property name="femur_width"  value="0.059"/>
   <xacro:property name="femur_height" value="0.020"/>
-  <xacro:property name="tibia_length" value="0.1787"/>
+  <xacro:property name="tibia_length" value="0.200"/>
   <xacro:property name="tibia_width"  value="0.012"/>
   <xacro:property name="tibia_height" value="0.012"/>
