Commit message: phase 9 stage F done

File: src/hexapod_description/urdf/hexapod.ros2_control.xacro (robot description, xacro)
@@ -2,17 +2,39 @@
 <robot xmlns:xacro="http://www.ros.org/wiki/xacro">
   <!--
-    ros2_control-Anbindung fuer die 18 Bein-Joints + gz_ros2_control-Plugin.
-    Wird vom robot_state_publisher ignoriert (auf dem Pi unschaedlich).
-    Phase 7 ersetzt das gz_ros2_control-Plugin durch ein Custom-
-    HardwareInterface fuer die Servo2040; controllers.yaml und
-    Interface-Deklarationen bleiben dabei unveraendert.
+    ros2_control-Anbindung fuer die 18 Bein-Joints.
+    Sim/HW-Switch (Phase 9 Stufe F): das Argument `use_sim` (Top-Level-
+    Default true) waehlt zwischen
+      - gz_ros2_control/GazeboSimSystem  (Phase 4-6, Sim-Pfad)
+      - hexapod_hardware/HexapodSystemHardware (Phase 9, echte Servo2040)
+    Die Wahl ist mutually exclusive — beide Plugins koennen nicht
+    gleichzeitig denselben Joint-Pool besitzen (ros2_control-Constraint).
+    Hardware-Parameter (`serial_port`, `loopback_mode`) werden nur im
+    HW-Pfad evaluiert, sind aber im Top-File ebenfalls als <xacro:arg>
+    deklariert (siehe hexapod.urdf.xacro), damit Launch-Files sie
+    sauber als oeffentliches Interface ueberschreiben koennen ohne
+    den Include zu kennen. Defaults: /dev/ttyACM0 + loopback_mode=false.
+    Velocity-State-Interface ist nur im Sim-Pfad exportiert. Gazebo's
+    GazeboSimSystem liefert echtes Velocity-Feedback; das Servo2040-
+    Plugin hat strukturell kein Velocity-Feedback (Echo-State, siehe
+    hexapod_hardware/README.md). controllers.real.yaml listet daher
+    nur position-state, controllers.yaml weiterhin position+velocity.
     Limit-Werte stammen aus hexapod_physical_properties.xacro
     (Single Source of Truth, siehe 00_conventions.md §11.4).
     Doppeltes Sicherheitsnetz: controller_manager clamped auf
-    <param min/max>, Gazebo zusaetzlich auf <limit>.
+    <param min/max>, Gazebo zusaetzlich auf <limit>, Plugin zusaetzlich
+    auf Calibration::set_joint_limits-Strikt-Range-Check.
   -->
+  <xacro:property name="use_sim" value="$(arg use_sim)"/>
   <ros2_control name="GazeboSimSystem" type="system">
     <hardware>
-      <plugin>gz_ros2_control/GazeboSimSystem</plugin>
+      <xacro:if value="${use_sim}">
+        <plugin>gz_ros2_control/GazeboSimSystem</plugin>
+      </xacro:if>
+      <xacro:unless value="${use_sim}">
+        <plugin>hexapod_hardware/HexapodSystemHardware</plugin>
+        <param name="serial_port">$(arg serial_port)</param>
+        <param name="calibration_file">$(find hexapod_hardware)/config/servo_mapping.yaml</param>
+        <param name="loopback_mode">$(arg loopback_mode)</param>
+      </xacro:unless>
     </hardware>
     <xacro:macro name="joint_iface" params="name lower upper">
@@ -23,5 +45,7 @@
         </command_interface>
         <state_interface name="position"/>
-        <state_interface name="velocity"/>
+        <xacro:if value="${use_sim}">
+          <state_interface name="velocity"/>
+        </xacro:if>
       </joint>
     </xacro:macro>
@@ -52,13 +76,18 @@
   </ros2_control>
   <!--
-    gz_ros2_control-System-Plugin: laedt controllers.yaml und startet
-    den controller_manager im Sim-Prozess. $(find ...) wird von xacro
-    aufgeloest, daher muss hexapod_control vorher gebaut + gesourct sein.
+    Gazebo-System-Plugin: laedt controllers.yaml und startet den
+    controller_manager im Sim-Prozess. Nur im Sim-Pfad relevant — im
+    HW-Pfad startet ros2_control_node aus real.launch.py (Stage G)
+    den controller_manager mit controllers.real.yaml separat.
+    $(find ...) wird von xacro aufgeloest, daher muss hexapod_control
+    vorher gebaut + gesourct sein.
   -->
-  <gazebo>
-    <plugin filename="gz_ros2_control-system"
-            name="gz_ros2_control::GazeboSimROS2ControlPlugin">
-      <parameters>$(find hexapod_control)/config/controllers.yaml</parameters>
-    </plugin>
-  </gazebo>
+  <xacro:if value="${use_sim}">
+    <gazebo>
+      <plugin filename="gz_ros2_control-system"
+              name="gz_ros2_control::GazeboSimROS2ControlPlugin">
+        <parameters>$(find hexapod_control)/config/controllers.yaml</parameters>
+      </plugin>
+    </gazebo>
+  </xacro:if>
 </robot>

File: src/hexapod_description/urdf/hexapod.urdf.xacro (robot description, xacro)
@@ -6,4 +6,23 @@
        gestartet (siehe hexapod_bringup/launch/sim.launch.py). -->
   <xacro:arg name="enable_foot_contact" default="true"/>
+  <!-- Phase 9 Stufe F: Sim/HW-Switch + Hardware-Parameter.
+       Diese drei Args sind die "öffentliche Schnittstelle" des URDF-
+       Moduls für Phase 9. Konsumiert werden sie in
+       hexapod.ros2_control.xacro (xacro:if-Branches und <param>-Werte
+       im hexapod_hardware-Plugin), aber sie sind hier im Top-File
+       deklariert, damit:
+         (1) sie an einer Stelle dokumentiert sind ("welche Args nimmt
+             dieses URDF entgegen?"),
+         (2) ein Refactor des Includes (z.B. conditional include in
+             einer späteren Stage) die Arg-Deklaration nicht still
+             entfernt,
+         (3) striktere künftige xacro-Versionen, die alle CLI-Args im
+             Top-File deklariert sehen wollen, sauber funktionieren.
+       Konvention konsistent mit `enable_foot_contact` oben.
+       Defaults sind Sim-kompatibel — `xacro hexapod.urdf.xacro`
+       ohne Args ergibt 1:1 das Pre-Phase-9-URDF. -->
+  <xacro:arg name="use_sim" default="true"/>
+  <xacro:arg name="serial_port" default="/dev/ttyACM0"/>
+  <xacro:arg name="loopback_mode" default="false"/>
   <xacro:include filename="hexapod_physical_properties.xacro"/>
   <xacro:include filename="materials.xacro"/>

Commit message: 18 per-Bein-rad-Werte (PWM-zentrisch) sowohl in <limit>-Tags (via leg.xacro args) als auch in ros2_control <param min/max> eingetragen. Plugin-Fix aus Stage 0 macht direction-Spiegelung transparent → keine Werte-Spiegelung nötig.
Beifang: hexapod.ros2_control.xacro war in Stage A nicht refactored
(Macro-Aufrufer nutzten globale -Properties statt per-Bein).
Jetzt analog zu leg.xacro per-Bein-Werte.

File: src/hexapod_description/urdf/hexapod.ros2_control.xacro (robot description, xacro)
@@ -50,28 +50,32 @@
       </joint>
     </xacro:macro>
-    <!-- Bein 1 -->
-    <xacro:joint_iface name="leg_1_coxa_joint"  lower="${coxa_lower}"  upper="${coxa_upper}"/>
-    <xacro:joint_iface name="leg_1_femur_joint" lower="${femur_lower}" upper="${femur_upper}"/>
-    <xacro:joint_iface name="leg_1_tibia_joint" lower="${tibia_lower}" upper="${tibia_upper}"/>
-    <!-- Bein 2 -->
-    <xacro:joint_iface name="leg_2_coxa_joint"  lower="${coxa_lower}"  upper="${coxa_upper}"/>
-    <xacro:joint_iface name="leg_2_femur_joint" lower="${femur_lower}" upper="${femur_upper}"/>
-    <xacro:joint_iface name="leg_2_tibia_joint" lower="${tibia_lower}" upper="${tibia_upper}"/>
-    <!-- Bein 3 -->
-    <xacro:joint_iface name="leg_3_coxa_joint"  lower="${coxa_lower}"  upper="${coxa_upper}"/>
-    <xacro:joint_iface name="leg_3_femur_joint" lower="${femur_lower}" upper="${femur_upper}"/>
-    <xacro:joint_iface name="leg_3_tibia_joint" lower="${tibia_lower}" upper="${tibia_upper}"/>
-    <!-- Bein 4 -->
-    <xacro:joint_iface name="leg_4_coxa_joint"  lower="${coxa_lower}"  upper="${coxa_upper}"/>
-    <xacro:joint_iface name="leg_4_femur_joint" lower="${femur_lower}" upper="${femur_upper}"/>
-    <xacro:joint_iface name="leg_4_tibia_joint" lower="${tibia_lower}" upper="${tibia_upper}"/>
-    <!-- Bein 5 -->
-    <xacro:joint_iface name="leg_5_coxa_joint"  lower="${coxa_lower}"  upper="${coxa_upper}"/>
-    <xacro:joint_iface name="leg_5_femur_joint" lower="${femur_lower}" upper="${femur_upper}"/>
-    <xacro:joint_iface name="leg_5_tibia_joint" lower="${tibia_lower}" upper="${tibia_upper}"/>
-    <!-- Bein 6 -->
-    <xacro:joint_iface name="leg_6_coxa_joint"  lower="${coxa_lower}"  upper="${coxa_upper}"/>
-    <xacro:joint_iface name="leg_6_femur_joint" lower="${femur_lower}" upper="${femur_upper}"/>
-    <xacro:joint_iface name="leg_6_tibia_joint" lower="${tibia_lower}" upper="${tibia_upper}"/>
+    <!-- Stage D: per-Joint-Limits aus servo_real_calibration_todos.md
+         Tab. 3.3 (PWM-zentrisch, identisch zu den <limit>-Werten in den
+         <joint>-Tags via leg.xacro). Plugin liest diese als <param min/max>
+         und validiert via Calibration::set_joint_limits. -->
+    <!-- Bein 1 (front-right) -->
+    <xacro:joint_iface name="leg_1_coxa_joint"  lower="-0.747" upper="0.569"/>
+    <xacro:joint_iface name="leg_1_femur_joint" lower="-1.529" upper="1.564"/>
+    <xacro:joint_iface name="leg_1_tibia_joint" lower="-1.920" upper="1.197"/>
+    <!-- Bein 2 (mid-right) -->
+    <xacro:joint_iface name="leg_2_coxa_joint"  lower="-0.474" upper="0.415"/>
+    <xacro:joint_iface name="leg_2_femur_joint" lower="-1.588" upper="1.517"/>
+    <xacro:joint_iface name="leg_2_tibia_joint" lower="-1.943" upper="1.232"/>
+    <!-- Bein 3 (back-right) -->
+    <xacro:joint_iface name="leg_3_coxa_joint"  lower="-0.498" upper="0.794"/>
+    <xacro:joint_iface name="leg_3_femur_joint" lower="-1.529" upper="1.553"/>
+    <xacro:joint_iface name="leg_3_tibia_joint" lower="-1.967" upper="1.185"/>
+    <!-- Bein 4 (back-left) -->
+    <xacro:joint_iface name="leg_4_coxa_joint"  lower="-0.758" upper="0.427"/>
+    <xacro:joint_iface name="leg_4_femur_joint" lower="-1.636" upper="1.493"/>
+    <xacro:joint_iface name="leg_4_tibia_joint" lower="-1.197" upper="1.943"/>
+    <!-- Bein 5 (mid-left) -->
+    <xacro:joint_iface name="leg_5_coxa_joint"  lower="-0.474" upper="0.474"/>
+    <xacro:joint_iface name="leg_5_femur_joint" lower="-1.588" upper="1.564"/>
+    <xacro:joint_iface name="leg_5_tibia_joint" lower="-1.197" upper="1.943"/>
+    <!-- Bein 6 (front-left) -->
+    <xacro:joint_iface name="leg_6_coxa_joint"  lower="-0.569" upper="0.806"/>
+    <xacro:joint_iface name="leg_6_femur_joint" lower="-1.659" upper="1.493"/>
+    <xacro:joint_iface name="leg_6_tibia_joint" lower="-1.161" upper="1.967"/>
   </ros2_control>
   <!--

File: src/hexapod_description/urdf/hexapod.urdf.xacro (robot description, xacro)
@@ -45,23 +45,45 @@
                        x="${body_length}" y="${body_width}" z="${body_height}"/>
   </link>
-  <!-- ===== Beine (Mountpunkte + yaw aus 00_conventions.md §11.3) ===== -->
+  <!-- ===== Beine (Mountpunkte + yaw aus 00_conventions.md §11.3) =====
+       Stage D: per-Bein-Joint-Limits aus servo_real_calibration_todos.md
+       Tab. 3.3 (PWM-zentrisch, dank Stage-0-Plugin-Fix keine Spiegelung
+       für direction=-1 nötig). Werte aus Cal-Session 2026-05-21 +
+       leg_2/leg_5 re-cal 2026-05-24 nach Mount-Tausch. -->
   <xacro:leg id="1"
              mount_x="${ body_length/2}" mount_y="${-body_width/2}"
-             mount_z="${leg_mount_z}"    mount_yaw="${-pi/4}"/>
+             mount_z="${leg_mount_z}"    mount_yaw="${-pi/4}"
+             coxa_lower="-0.747"  coxa_upper="0.569"
+             femur_lower="-1.529" femur_upper="1.564"
+             tibia_lower="-1.920" tibia_upper="1.197"/>
   <xacro:leg id="2"
              mount_x="0"                 mount_y="${-body_width_middle/2}"
-             mount_z="${leg_mount_z}"    mount_yaw="${-pi/2}"/>
+             mount_z="${leg_mount_z}"    mount_yaw="${-pi/2}"
+             coxa_lower="-0.474"  coxa_upper="0.415"
+             femur_lower="-1.588" femur_upper="1.517"
+             tibia_lower="-1.943" tibia_upper="1.232"/>
   <xacro:leg id="3"
              mount_x="${-body_length/2}" mount_y="${-body_width/2}"
-             mount_z="${leg_mount_z}"    mount_yaw="${-3*pi/4}"/>
+             mount_z="${leg_mount_z}"    mount_yaw="${-3*pi/4}"
+             coxa_lower="-0.498"  coxa_upper="0.794"
+             femur_lower="-1.529" femur_upper="1.553"
+             tibia_lower="-1.967" tibia_upper="1.185"/>
   <xacro:leg id="4"
              mount_x="${-body_length/2}" mount_y="${ body_width/2}"
-             mount_z="${leg_mount_z}"    mount_yaw="${ 3*pi/4}"/>
+             mount_z="${leg_mount_z}"    mount_yaw="${ 3*pi/4}"
+             coxa_lower="-0.758"  coxa_upper="0.427"
+             femur_lower="-1.636" femur_upper="1.493"
+             tibia_lower="-1.197" tibia_upper="1.943"/>
   <xacro:leg id="5"
              mount_x="0"                 mount_y="${ body_width_middle/2}"
-             mount_z="${leg_mount_z}"    mount_yaw="${ pi/2}"/>
+             mount_z="${leg_mount_z}"    mount_yaw="${ pi/2}"
+             coxa_lower="-0.474"  coxa_upper="0.474"
+             femur_lower="-1.588" femur_upper="1.564"
+             tibia_lower="-1.197" tibia_upper="1.943"/>
   <xacro:leg id="6"
              mount_x="${ body_length/2}" mount_y="${ body_width/2}"
-             mount_z="${leg_mount_z}"    mount_yaw="${ pi/4}"/>
+             mount_z="${leg_mount_z}"    mount_yaw="${ pi/4}"
+             coxa_lower="-0.569"  coxa_upper="0.806"
+             femur_lower="-1.659" femur_upper="1.493"
+             tibia_lower="-1.161" tibia_upper="1.967"/>
   <!-- ===== Gazebo-spezifische Eigenschaften (Reibung an Foot-Kugeln) ===== -->
   <xacro:include filename="hexapod.gazebo.xacro"/>

Commit message: stage F of calibration done, roboter is walking on testbench

File: src/hexapod_description/urdf/hexapod.ros2_control.xacro (robot description, xacro)
@@ -50,32 +50,35 @@
       </joint>
     </xacro:macro>
-    <!-- Stage D: per-Joint-Limits aus servo_real_calibration_todos.md
-         Tab. 3.3 (PWM-zentrisch, identisch zu den <limit>-Werten in den
-         <joint>-Tags via leg.xacro). Plugin liest diese als <param min/max>
-         und validiert via Calibration::set_joint_limits. -->
+    <!-- Stage F (2026-05-25): rad-Limits strict-symmetrisch fuer alle
+         6 Beine identisch (coxa ±0.415 / femur ±1.493 / tibia ±1.161).
+         Behebt visuelle Asymmetrie aus Stage E2.3 — siehe
+         docs_raspi/servo_real_cal_stage_f_urdf_symmetrize_plan.md.
+         Werte sind synchron zu hexapod.urdf.xacro <xacro:leg ...>-
+         Aufrufen. Plugin liest diese als <param min/max> und validiert
+         via Calibration::set_joint_limits. -->
     <!-- Bein 1 (front-right) -->
-    <xacro:joint_iface name="leg_1_coxa_joint"  lower="-0.747" upper="0.569"/>
-    <xacro:joint_iface name="leg_1_femur_joint" lower="-1.529" upper="1.564"/>
-    <xacro:joint_iface name="leg_1_tibia_joint" lower="-1.920" upper="1.197"/>
+    <xacro:joint_iface name="leg_1_coxa_joint"  lower="-0.415" upper="0.415"/>
+    <xacro:joint_iface name="leg_1_femur_joint" lower="-1.493" upper="1.493"/>
+    <xacro:joint_iface name="leg_1_tibia_joint" lower="-1.161" upper="1.161"/>
     <!-- Bein 2 (mid-right) -->
-    <xacro:joint_iface name="leg_2_coxa_joint"  lower="-0.474" upper="0.415"/>
-    <xacro:joint_iface name="leg_2_femur_joint" lower="-1.588" upper="1.517"/>
-    <xacro:joint_iface name="leg_2_tibia_joint" lower="-1.943" upper="1.232"/>
+    <xacro:joint_iface name="leg_2_coxa_joint"  lower="-0.415" upper="0.415"/>
+    <xacro:joint_iface name="leg_2_femur_joint" lower="-1.493" upper="1.493"/>
+    <xacro:joint_iface name="leg_2_tibia_joint" lower="-1.161" upper="1.161"/>
     <!-- Bein 3 (back-right) -->
-    <xacro:joint_iface name="leg_3_coxa_joint"  lower="-0.498" upper="0.794"/>
-    <xacro:joint_iface name="leg_3_femur_joint" lower="-1.529" upper="1.553"/>
-    <xacro:joint_iface name="leg_3_tibia_joint" lower="-1.967" upper="1.185"/>
+    <xacro:joint_iface name="leg_3_coxa_joint"  lower="-0.415" upper="0.415"/>
+    <xacro:joint_iface name="leg_3_femur_joint" lower="-1.493" upper="1.493"/>
+    <xacro:joint_iface name="leg_3_tibia_joint" lower="-1.161" upper="1.161"/>
     <!-- Bein 4 (back-left) -->
-    <xacro:joint_iface name="leg_4_coxa_joint"  lower="-0.758" upper="0.427"/>
-    <xacro:joint_iface name="leg_4_femur_joint" lower="-1.636" upper="1.493"/>
-    <xacro:joint_iface name="leg_4_tibia_joint" lower="-1.197" upper="1.943"/>
+    <xacro:joint_iface name="leg_4_coxa_joint"  lower="-0.415" upper="0.415"/>
+    <xacro:joint_iface name="leg_4_femur_joint" lower="-1.493" upper="1.493"/>
+    <xacro:joint_iface name="leg_4_tibia_joint" lower="-1.161" upper="1.161"/>
     <!-- Bein 5 (mid-left) -->
-    <xacro:joint_iface name="leg_5_coxa_joint"  lower="-0.474" upper="0.474"/>
-    <xacro:joint_iface name="leg_5_femur_joint" lower="-1.588" upper="1.564"/>
-    <xacro:joint_iface name="leg_5_tibia_joint" lower="-1.197" upper="1.943"/>
+    <xacro:joint_iface name="leg_5_coxa_joint"  lower="-0.415" upper="0.415"/>
+    <xacro:joint_iface name="leg_5_femur_joint" lower="-1.493" upper="1.493"/>
+    <xacro:joint_iface name="leg_5_tibia_joint" lower="-1.161" upper="1.161"/>
     <!-- Bein 6 (front-left) -->
-    <xacro:joint_iface name="leg_6_coxa_joint"  lower="-0.569" upper="0.806"/>
-    <xacro:joint_iface name="leg_6_femur_joint" lower="-1.659" upper="1.493"/>
-    <xacro:joint_iface name="leg_6_tibia_joint" lower="-1.161" upper="1.967"/>
+    <xacro:joint_iface name="leg_6_coxa_joint"  lower="-0.415" upper="0.415"/>
+    <xacro:joint_iface name="leg_6_femur_joint" lower="-1.493" upper="1.493"/>
+    <xacro:joint_iface name="leg_6_tibia_joint" lower="-1.161" upper="1.161"/>
   </ros2_control>
   <!--

File: src/hexapod_description/urdf/hexapod.urdf.xacro (robot description, xacro)
@@ -46,44 +46,50 @@
   </link>
   <!-- ===== Beine (Mountpunkte + yaw aus 00_conventions.md §11.3) =====
-       Stage D: per-Bein-Joint-Limits aus servo_real_calibration_todos.md
-       Tab. 3.3 (PWM-zentrisch, dank Stage-0-Plugin-Fix keine Spiegelung
-       für direction=-1 nötig). Werte aus Cal-Session 2026-05-21 +
-       leg_2/leg_5 re-cal 2026-05-24 nach Mount-Tausch. -->
+       Stage F (2026-05-25): rad-Limits strict-symmetrisch für alle 6
+       Beine identisch (coxa ±0.415 / femur ±1.493 / tibia ±1.161) —
+       behebt die in Stage E2.3 entdeckte visuelle Asymmetrie rechts/
+       links während Walking. Hintergrund: Plugin-Slope-Formel skaliert
+       rad→pulse über joint_lower/upper; per-Bein-Asymmetrie aus Stage D
+       erzeugte ~28° physische Differenz im Tibia. Werte = strict-min
+       der gemeinsamen Range (kleinster |lower|/upper aller 6 Beine pro
+       Joint-Typ). Siehe docs_raspi/servo_real_cal_stage_f_urdf_symmetrize_plan.md.
+       Vorherige Stage D-Werte (per-Bein-asymmetrisch, archiviert in
+       git-Historie): leg_1 tibia +1.197 vs leg_4 tibia +1.943 etc. -->
   <xacro:leg id="1"
              mount_x="${ body_length/2}" mount_y="${-body_width/2}"
              mount_z="${leg_mount_z}"    mount_yaw="${-pi/4}"
-             coxa_lower="-0.747"  coxa_upper="0.569"
-             femur_lower="-1.529" femur_upper="1.564"
-             tibia_lower="-1.920" tibia_upper="1.197"/>
+             coxa_lower="-0.415"  coxa_upper="0.415"
+             femur_lower="-1.493" femur_upper="1.493"
+             tibia_lower="-1.161" tibia_upper="1.161"/>
   <xacro:leg id="2"
              mount_x="0"                 mount_y="${-body_width_middle/2}"
              mount_z="${leg_mount_z}"    mount_yaw="${-pi/2}"
-             coxa_lower="-0.474"  coxa_upper="0.415"
-             femur_lower="-1.588" femur_upper="1.517"
-             tibia_lower="-1.943" tibia_upper="1.232"/>
+             coxa_lower="-0.415"  coxa_upper="0.415"
+             femur_lower="-1.493" femur_upper="1.493"
+             tibia_lower="-1.161" tibia_upper="1.161"/>
   <xacro:leg id="3"
              mount_x="${-body_length/2}" mount_y="${-body_width/2}"
              mount_z="${leg_mount_z}"    mount_yaw="${-3*pi/4}"
-             coxa_lower="-0.498"  coxa_upper="0.794"
-             femur_lower="-1.529" femur_upper="1.553"
-             tibia_lower="-1.967" tibia_upper="1.185"/>
+             coxa_lower="-0.415"  coxa_upper="0.415"
+             femur_lower="-1.493" femur_upper="1.493"
+             tibia_lower="-1.161" tibia_upper="1.161"/>
   <xacro:leg id="4"
              mount_x="${-body_length/2}" mount_y="${ body_width/2}"
              mount_z="${leg_mount_z}"    mount_yaw="${ 3*pi/4}"
-             coxa_lower="-0.758"  coxa_upper="0.427"
-             femur_lower="-1.636" femur_upper="1.493"
-             tibia_lower="-1.197" tibia_upper="1.943"/>
+             coxa_lower="-0.415"  coxa_upper="0.415"
+             femur_lower="-1.493" femur_upper="1.493"
+             tibia_lower="-1.161" tibia_upper="1.161"/>
   <xacro:leg id="5"
              mount_x="0"                 mount_y="${ body_width_middle/2}"
              mount_z="${leg_mount_z}"    mount_yaw="${ pi/2}"
-             coxa_lower="-0.474"  coxa_upper="0.474"
-             femur_lower="-1.588" femur_upper="1.564"
-             tibia_lower="-1.197" tibia_upper="1.943"/>
+             coxa_lower="-0.415"  coxa_upper="0.415"
+             femur_lower="-1.493" femur_upper="1.493"
+             tibia_lower="-1.161" tibia_upper="1.161"/>
   <xacro:leg id="6"
              mount_x="${ body_length/2}" mount_y="${ body_width/2}"
              mount_z="${leg_mount_z}"    mount_yaw="${ pi/4}"
-             coxa_lower="-0.569"  coxa_upper="0.806"
-             femur_lower="-1.659" femur_upper="1.493"
-             tibia_lower="-1.161" tibia_upper="1.967"/>
+             coxa_lower="-0.415"  coxa_upper="0.415"
+             femur_lower="-1.493" femur_upper="1.493"
+             tibia_lower="-1.161" tibia_upper="1.161"/>
   <!-- ===== Gazebo-spezifische Eigenschaften (Reibung an Foot-Kugeln) ===== -->
   <xacro:include filename="hexapod.gazebo.xacro"/>
