Commit message: phase 13 stage 0.5 done, aber fuesser schrammen am boden etwas nach innen beim aufstehen, muss untersucht werden

File: src/hexapod_description/urdf/hexapod.ros2_control.xacro (robot description, xacro)
@@ -41,5 +41,18 @@
       </xacro:unless>
     </hardware>
-    <xacro:macro name="joint_iface" params="name lower upper">
+    <!--
+      Phase 13 Stage 0.5: `initial` (rad) = power_on_mid-Startwinkel des
+      Joints. NUR im Sim-Pfad als <param name="initial_value"> am position-
+      state_interface gesetzt → gz_ros2_control spawnt den Joint bei diesem
+      Winkel statt bei 0 (T-Pose). So startet die Sim in genau der Pose, die
+      die echte HW nach dem Servo2040-Init (1500 µs) meldet, und steht von
+      dort mit der 0.4-STARTUP_RAMP auf.
+      HW-sicher: im <xacro:unless use_sim>-Zweig bleibt das position-
+      state_interface nackt — das HW-Plugin liest `initial_value` nie.
+      Werte = _POWER_ON_MID aus hexapod_gait/test/test_startup_ramp.py
+      (Quelle: phase_13_stage_0_4_standup_plan.md §3.1). Bei Neu-Cal der
+      Femurs nachziehen.
+    -->
+    <xacro:macro name="joint_iface" params="name lower upper initial:=0.0">
       <joint name="${name}">
         <command_interface name="position">
@@ -47,8 +60,13 @@
           <param name="max">${upper}</param>
         </command_interface>
-        <state_interface name="position"/>
         <xacro:if value="${use_sim}">
+          <state_interface name="position">
+            <param name="initial_value">${initial}</param>
+          </state_interface>
           <state_interface name="velocity"/>
         </xacro:if>
+        <xacro:unless value="${use_sim}">
+          <state_interface name="position"/>
+        </xacro:unless>
       </joint>
     </xacro:macro>
@@ -62,27 +80,27 @@
          via Calibration::set_joint_limits. -->
     <!-- Bein 1 (front-right) -->
-    <xacro:joint_iface name="leg_1_coxa_joint"  lower="-0.415" upper="0.415"/>
-    <xacro:joint_iface name="leg_1_femur_joint" lower="-1.57" upper="1.57"/>
-    <xacro:joint_iface name="leg_1_tibia_joint" lower="-1.161" upper="1.161"/>
+    <xacro:joint_iface name="leg_1_coxa_joint"  lower="-0.415" upper="0.415" initial="-0.069"/>
+    <xacro:joint_iface name="leg_1_femur_joint" lower="-1.57" upper="1.57" initial="-0.469"/>
+    <xacro:joint_iface name="leg_1_tibia_joint" lower="-1.161" upper="1.161" initial="0.258"/>
     <!-- Bein 2 (mid-right) -->
-    <xacro:joint_iface name="leg_2_coxa_joint"  lower="-0.415" upper="0.415"/>
-    <xacro:joint_iface name="leg_2_femur_joint" lower="-1.57" upper="1.57"/>
-    <xacro:joint_iface name="leg_2_tibia_joint" lower="-1.161" upper="1.161"/>
+    <xacro:joint_iface name="leg_2_coxa_joint"  lower="-0.415" upper="0.415" initial="0.156"/>
+    <xacro:joint_iface name="leg_2_femur_joint" lower="-1.57" upper="1.57" initial="-0.637"/>
+    <xacro:joint_iface name="leg_2_tibia_joint" lower="-1.161" upper="1.161" initial="0.255"/>
     <!-- Bein 3 (back-right) -->
-    <xacro:joint_iface name="leg_3_coxa_joint"  lower="-0.415" upper="0.415"/>
-    <xacro:joint_iface name="leg_3_femur_joint" lower="-1.57" upper="1.57"/>
-    <xacro:joint_iface name="leg_3_tibia_joint" lower="-1.161" upper="1.161"/>
+    <xacro:joint_iface name="leg_3_coxa_joint"  lower="-0.415" upper="0.415" initial="-0.111"/>
+    <xacro:joint_iface name="leg_3_femur_joint" lower="-1.57" upper="1.57" initial="-0.439"/>
+    <xacro:joint_iface name="leg_3_tibia_joint" lower="-1.161" upper="1.161" initial="0.168"/>
     <!-- Bein 4 (back-left) -->
-    <xacro:joint_iface name="leg_4_coxa_joint"  lower="-0.415" upper="0.415"/>
-    <xacro:joint_iface name="leg_4_femur_joint" lower="-1.57" upper="1.57"/>
-    <xacro:joint_iface name="leg_4_tibia_joint" lower="-1.161" upper="1.161"/>
+    <xacro:joint_iface name="leg_4_coxa_joint"  lower="-0.415" upper="0.415" initial="0.026"/>
+    <xacro:joint_iface name="leg_4_femur_joint" lower="-1.57" upper="1.57" initial="-0.477"/>
+    <xacro:joint_iface name="leg_4_tibia_joint" lower="-1.161" upper="1.161" initial="0.255"/>
     <!-- Bein 5 (mid-left) -->
-    <xacro:joint_iface name="leg_5_coxa_joint"  lower="-0.415" upper="0.415"/>
-    <xacro:joint_iface name="leg_5_femur_joint" lower="-1.57" upper="1.57"/>
-    <xacro:joint_iface name="leg_5_tibia_joint" lower="-1.161" upper="1.161"/>
+    <xacro:joint_iface name="leg_5_coxa_joint"  lower="-0.415" upper="0.415" initial="0.104"/>
+    <xacro:joint_iface name="leg_5_femur_joint" lower="-1.57" upper="1.57" initial="-0.419"/>
+    <xacro:joint_iface name="leg_5_tibia_joint" lower="-1.161" upper="1.161" initial="0.156"/>
     <!-- Bein 6 (front-left) -->
-    <xacro:joint_iface name="leg_6_coxa_joint"  lower="-0.415" upper="0.415"/>
-    <xacro:joint_iface name="leg_6_femur_joint" lower="-1.57" upper="1.57"/>
-    <xacro:joint_iface name="leg_6_tibia_joint" lower="-1.161" upper="1.161"/>
+    <xacro:joint_iface name="leg_6_coxa_joint"  lower="-0.415" upper="0.415" initial="0.052"/>
+    <xacro:joint_iface name="leg_6_femur_joint" lower="-1.57" upper="1.57" initial="-0.496"/>
+    <xacro:joint_iface name="leg_6_tibia_joint" lower="-1.161" upper="1.161" initial="0.224"/>
   </ros2_control>
   <!--

Commit message: phase 13 stage 0.6 done, hexapod can stand up and walk, but need some improvements

File: src/hexapod_description/urdf/hexapod.ros2_control.xacro (robot description, xacro)
@@ -82,25 +82,25 @@
     <xacro:joint_iface name="leg_1_coxa_joint"  lower="-0.415" upper="0.415" initial="-0.069"/>
     <xacro:joint_iface name="leg_1_femur_joint" lower="-1.57" upper="1.57" initial="-0.469"/>
-    <xacro:joint_iface name="leg_1_tibia_joint" lower="-1.161" upper="1.161" initial="0.258"/>
+    <xacro:joint_iface name="leg_1_tibia_joint" lower="-1.00" upper="1.30" initial="0.4946"/>
     <!-- Bein 2 (mid-right) -->
     <xacro:joint_iface name="leg_2_coxa_joint"  lower="-0.415" upper="0.415" initial="0.156"/>
     <xacro:joint_iface name="leg_2_femur_joint" lower="-1.57" upper="1.57" initial="-0.637"/>
-    <xacro:joint_iface name="leg_2_tibia_joint" lower="-1.161" upper="1.161" initial="0.255"/>
+    <xacro:joint_iface name="leg_2_tibia_joint" lower="-1.00" upper="1.30" initial="0.5181"/>
     <!-- Bein 3 (back-right) -->
     <xacro:joint_iface name="leg_3_coxa_joint"  lower="-0.415" upper="0.415" initial="-0.111"/>
     <xacro:joint_iface name="leg_3_femur_joint" lower="-1.57" upper="1.57" initial="-0.439"/>
-    <xacro:joint_iface name="leg_3_tibia_joint" lower="-1.161" upper="1.161" initial="0.168"/>
+    <xacro:joint_iface name="leg_3_tibia_joint" lower="-1.00" upper="1.30" initial="0.2591"/>
     <!-- Bein 4 (back-left) -->
     <xacro:joint_iface name="leg_4_coxa_joint"  lower="-0.415" upper="0.415" initial="0.026"/>
     <xacro:joint_iface name="leg_4_femur_joint" lower="-1.57" upper="1.57" initial="-0.477"/>
-    <xacro:joint_iface name="leg_4_tibia_joint" lower="-1.161" upper="1.161" initial="0.255"/>
+    <xacro:joint_iface name="leg_4_tibia_joint" lower="-1.00" upper="1.30" initial="0.4286"/>
     <!-- Bein 5 (mid-left) -->
     <xacro:joint_iface name="leg_5_coxa_joint"  lower="-0.415" upper="0.415" initial="0.104"/>
     <xacro:joint_iface name="leg_5_femur_joint" lower="-1.57" upper="1.57" initial="-0.419"/>
-    <xacro:joint_iface name="leg_5_tibia_joint" lower="-1.161" upper="1.161" initial="0.156"/>
+    <xacro:joint_iface name="leg_5_tibia_joint" lower="-1.00" upper="1.30" initial="0.1978"/>
     <!-- Bein 6 (front-left) -->
     <xacro:joint_iface name="leg_6_coxa_joint"  lower="-0.415" upper="0.415" initial="0.052"/>
     <xacro:joint_iface name="leg_6_femur_joint" lower="-1.57" upper="1.57" initial="-0.496"/>
-    <xacro:joint_iface name="leg_6_tibia_joint" lower="-1.161" upper="1.161" initial="0.224"/>
+    <xacro:joint_iface name="leg_6_tibia_joint" lower="-1.00" upper="1.30" initial="0.3503"/>
   </ros2_control>
   <!--

File: src/hexapod_description/urdf/hexapod.urdf.xacro (robot description, xacro)
@@ -62,5 +62,12 @@
        Joint-Typ). Siehe docs_raspi/servo_real_cal_stage_f_urdf_symmetrize_plan.md.
        Vorherige Stage D-Werte (per-Bein-asymmetrisch, archiviert in
-       git-Historie): leg_1 tibia +1.197 vs leg_4 tibia +1.943 etc. -->
+       git-Historie): leg_1 tibia +1.197 vs leg_4 tibia +1.943 etc.
+       Stage 0.6.6 (2026-06-01): Tibia jetzt ASYMMETRISCH -1.00 / +1.30
+       (global, alle 6 gleich). Begründung: die Tibia ist ein einseitiges
+       Knie — +rad (Beuge) wird voll genutzt (Standup/Walking bis +0.88),
+       -rad (Streck über gerade hinaus) NIE. Beuge +1.30 (74°, 24° Reserve
+       über Demand) / Streck -1.00 (innerhalb des mech. Anschlags ~58-72°).
+       Links/Rechts bleibt symmetrisch (Asymmetrie = Beuge≠Streck, analog
+       Femur DL-5). Cal: docs_raspi/phase_13_stage_0_6_6_tibia_recal_plan.md. -->
   <xacro:leg id="1"
              mount_x="${ body_length/2}" mount_y="${-body_width/2}"
@@ -68,5 +75,5 @@
              coxa_lower="-0.415"  coxa_upper="0.415"
              femur_lower="-1.57"  femur_upper="1.57"
-             tibia_lower="-1.161" tibia_upper="1.161"/>
+             tibia_lower="-1.00"  tibia_upper="1.30"/>
   <xacro:leg id="2"
              mount_x="0"                 mount_y="${-body_width_middle/2}"
@@ -74,5 +81,5 @@
              coxa_lower="-0.415"  coxa_upper="0.415"
              femur_lower="-1.57"  femur_upper="1.57"
-             tibia_lower="-1.161" tibia_upper="1.161"/>
+             tibia_lower="-1.00"  tibia_upper="1.30"/>
   <xacro:leg id="3"
              mount_x="${-body_length/2}" mount_y="${-body_width/2}"
@@ -80,5 +87,5 @@
              coxa_lower="-0.415"  coxa_upper="0.415"
              femur_lower="-1.57"  femur_upper="1.57"
-             tibia_lower="-1.161" tibia_upper="1.161"/>
+             tibia_lower="-1.00"  tibia_upper="1.30"/>
   <xacro:leg id="4"
              mount_x="${-body_length/2}" mount_y="${ body_width/2}"
@@ -86,5 +93,5 @@
              coxa_lower="-0.415"  coxa_upper="0.415"
              femur_lower="-1.57"  femur_upper="1.57"
-             tibia_lower="-1.161" tibia_upper="1.161"/>
+             tibia_lower="-1.00"  tibia_upper="1.30"/>
   <xacro:leg id="5"
              mount_x="0"                 mount_y="${ body_width_middle/2}"
@@ -92,5 +99,5 @@
              coxa_lower="-0.415"  coxa_upper="0.415"
              femur_lower="-1.57"  femur_upper="1.57"
-             tibia_lower="-1.161" tibia_upper="1.161"/>
+             tibia_lower="-1.00"  tibia_upper="1.30"/>
   <xacro:leg id="6"
              mount_x="${ body_length/2}" mount_y="${ body_width/2}"
@@ -98,5 +105,5 @@
              coxa_lower="-0.415"  coxa_upper="0.415"
              femur_lower="-1.57"  femur_upper="1.57"
-             tibia_lower="-1.161" tibia_upper="1.161"/>
+             tibia_lower="-1.00"  tibia_upper="1.30"/>
   <!-- ===== Gazebo-spezifische Eigenschaften (Reibung an Foot-Kugeln) ===== -->
   <xacro:include filename="hexapod.gazebo.xacro"/>

File: src/hexapod_description/urdf/hexapod_physical_properties.xacro (robot description, xacro)
@@ -26,6 +26,9 @@
   <xacro:property name="femur_lower"  value="-1.57"/>
   <xacro:property name="femur_upper"  value=" 1.57"/>
-  <xacro:property name="tibia_lower"  value="-1.50"/>
-  <xacro:property name="tibia_upper"  value=" 1.50"/>
+  <!-- Stage 0.6.6 (2026-06-01): Tibia asymmetrisch -1.00 / +1.30 (einseitiges
+       Knie). Spiegelt config.py::_TIBIA_LIMITS (Cross-Check test_config.py) und
+       die per-Bein-Overrides in hexapod.urdf.xacro. -->
+  <xacro:property name="tibia_lower"  value="-1.00"/>
+  <xacro:property name="tibia_upper"  value=" 1.30"/>
   <xacro:property name="joint_effort"   value="5.0"/>  <!-- effort/velocity: vom Servo-DB -->
   <xacro:property name="joint_velocity" value="2.0"/>

Commit message: phase 13 unlock full range of tibia, works in gazebo and real hw

File: src/hexapod_description/urdf/hexapod.ros2_control.xacro (robot description, xacro)
@@ -82,25 +82,25 @@
     <xacro:joint_iface name="leg_1_coxa_joint"  lower="-0.415" upper="0.415" initial="-0.069"/>
     <xacro:joint_iface name="leg_1_femur_joint" lower="-1.57" upper="1.57" initial="-0.469"/>
-    <xacro:joint_iface name="leg_1_tibia_joint" lower="-1.00" upper="1.30" initial="0.4946"/>
+    <xacro:joint_iface name="leg_1_tibia_joint" lower="-1.00" upper="2.50" initial="0.4946"/>
     <!-- Bein 2 (mid-right) -->
     <xacro:joint_iface name="leg_2_coxa_joint"  lower="-0.415" upper="0.415" initial="0.156"/>
     <xacro:joint_iface name="leg_2_femur_joint" lower="-1.57" upper="1.57" initial="-0.637"/>
-    <xacro:joint_iface name="leg_2_tibia_joint" lower="-1.00" upper="1.30" initial="0.5181"/>
+    <xacro:joint_iface name="leg_2_tibia_joint" lower="-1.00" upper="2.50" initial="0.5181"/>
     <!-- Bein 3 (back-right) -->
     <xacro:joint_iface name="leg_3_coxa_joint"  lower="-0.415" upper="0.415" initial="-0.111"/>
     <xacro:joint_iface name="leg_3_femur_joint" lower="-1.57" upper="1.57" initial="-0.439"/>
-    <xacro:joint_iface name="leg_3_tibia_joint" lower="-1.00" upper="1.30" initial="0.2591"/>
+    <xacro:joint_iface name="leg_3_tibia_joint" lower="-1.00" upper="2.50" initial="0.2591"/>
     <!-- Bein 4 (back-left) -->
     <xacro:joint_iface name="leg_4_coxa_joint"  lower="-0.415" upper="0.415" initial="0.026"/>
     <xacro:joint_iface name="leg_4_femur_joint" lower="-1.57" upper="1.57" initial="-0.477"/>
-    <xacro:joint_iface name="leg_4_tibia_joint" lower="-1.00" upper="1.30" initial="0.4286"/>
+    <xacro:joint_iface name="leg_4_tibia_joint" lower="-1.00" upper="2.50" initial="0.4286"/>
     <!-- Bein 5 (mid-left) -->
     <xacro:joint_iface name="leg_5_coxa_joint"  lower="-0.415" upper="0.415" initial="0.104"/>
     <xacro:joint_iface name="leg_5_femur_joint" lower="-1.57" upper="1.57" initial="-0.419"/>
-    <xacro:joint_iface name="leg_5_tibia_joint" lower="-1.00" upper="1.30" initial="0.1978"/>
+    <xacro:joint_iface name="leg_5_tibia_joint" lower="-1.00" upper="2.50" initial="0.1978"/>
     <!-- Bein 6 (front-left) -->
     <xacro:joint_iface name="leg_6_coxa_joint"  lower="-0.415" upper="0.415" initial="0.052"/>
     <xacro:joint_iface name="leg_6_femur_joint" lower="-1.57" upper="1.57" initial="-0.496"/>
-    <xacro:joint_iface name="leg_6_tibia_joint" lower="-1.00" upper="1.30" initial="0.3503"/>
+    <xacro:joint_iface name="leg_6_tibia_joint" lower="-1.00" upper="2.50" initial="0.3503"/>
   </ros2_control>
   <!--

File: src/hexapod_description/urdf/hexapod.urdf.xacro (robot description, xacro)
@@ -63,11 +63,13 @@
        Vorherige Stage D-Werte (per-Bein-asymmetrisch, archiviert in
        git-Historie): leg_1 tibia +1.197 vs leg_4 tibia +1.943 etc.
-       Stage 0.6.6 (2026-06-01): Tibia jetzt ASYMMETRISCH -1.00 / +1.30
-       (global, alle 6 gleich). Begründung: die Tibia ist ein einseitiges
-       Knie — +rad (Beuge) wird voll genutzt (Standup/Walking bis +0.88),
-       -rad (Streck über gerade hinaus) NIE. Beuge +1.30 (74°, 24° Reserve
-       über Demand) / Streck -1.00 (innerhalb des mech. Anschlags ~58-72°).
-       Links/Rechts bleibt symmetrisch (Asymmetrie = Beuge≠Streck, analog
-       Femur DL-5). Cal: docs_raspi/phase_13_stage_0_6_6_tibia_recal_plan.md. -->
+       Stage 1 / Teil 2.1 (2026-06-02): Tibia-Beuge auf Mechanik-Max
+       ASYMMETRISCH -1.00 / +2.50 freigeschaltet (war +1.30, konservativ).
+       Einseitiges Knie: +rad (Beuge) jetzt voll bis +2.50 (143°) nutzbar
+       für die feet-closer Lauf-Pose; -rad (Streck) bleibt -1.00 (nie genutzt).
+       +2.50 = strikt-symmetrisches Maximum, das ALLE 6 Servos puls-seitig
+       erreichen (leg_5-bound). Sicherheit pose-abhängig (Femur beim Laufen
+       oben) per Envelope-Check, kein Laufzeit-Kollisions-Check (Weg B deferred).
+       Cal-Modell: docs_raspi/phase_13_stage_0_6_6_tibia_recal_plan.md.
+       Unlock-Plan: docs_raspi/phase_13_stage_1_tibia_unlock_plan.md. -->
   <xacro:leg id="1"
              mount_x="${ body_length/2}" mount_y="${-body_width/2}"
@@ -75,5 +77,5 @@
              coxa_lower="-0.415"  coxa_upper="0.415"
              femur_lower="-1.57"  femur_upper="1.57"
-             tibia_lower="-1.00"  tibia_upper="1.30"/>
+             tibia_lower="-1.00"  tibia_upper="2.50"/>
   <xacro:leg id="2"
              mount_x="0"                 mount_y="${-body_width_middle/2}"
@@ -81,5 +83,5 @@
              coxa_lower="-0.415"  coxa_upper="0.415"
              femur_lower="-1.57"  femur_upper="1.57"
-             tibia_lower="-1.00"  tibia_upper="1.30"/>
+             tibia_lower="-1.00"  tibia_upper="2.50"/>
   <xacro:leg id="3"
              mount_x="${-body_length/2}" mount_y="${-body_width/2}"
@@ -87,5 +89,5 @@
              coxa_lower="-0.415"  coxa_upper="0.415"
              femur_lower="-1.57"  femur_upper="1.57"
-             tibia_lower="-1.00"  tibia_upper="1.30"/>
+             tibia_lower="-1.00"  tibia_upper="2.50"/>
   <xacro:leg id="4"
              mount_x="${-body_length/2}" mount_y="${ body_width/2}"
@@ -93,5 +95,5 @@
              coxa_lower="-0.415"  coxa_upper="0.415"
              femur_lower="-1.57"  femur_upper="1.57"
-             tibia_lower="-1.00"  tibia_upper="1.30"/>
+             tibia_lower="-1.00"  tibia_upper="2.50"/>
   <xacro:leg id="5"
              mount_x="0"                 mount_y="${ body_width_middle/2}"
@@ -99,5 +101,5 @@
              coxa_lower="-0.415"  coxa_upper="0.415"
              femur_lower="-1.57"  femur_upper="1.57"
-             tibia_lower="-1.00"  tibia_upper="1.30"/>
+             tibia_lower="-1.00"  tibia_upper="2.50"/>
   <xacro:leg id="6"
              mount_x="${ body_length/2}" mount_y="${ body_width/2}"
@@ -105,5 +107,5 @@
              coxa_lower="-0.415"  coxa_upper="0.415"
              femur_lower="-1.57"  femur_upper="1.57"
-             tibia_lower="-1.00"  tibia_upper="1.30"/>
+             tibia_lower="-1.00"  tibia_upper="2.50"/>
   <!-- ===== Gazebo-spezifische Eigenschaften (Reibung an Foot-Kugeln) ===== -->
   <xacro:include filename="hexapod.gazebo.xacro"/>

File: src/hexapod_description/urdf/hexapod_physical_properties.xacro (robot description, xacro)
@@ -26,9 +26,14 @@
   <xacro:property name="femur_lower"  value="-1.57"/>
   <xacro:property name="femur_upper"  value=" 1.57"/>
-  <!-- Stage 0.6.6 (2026-06-01): Tibia asymmetrisch -1.00 / +1.30 (einseitiges
-       Knie). Spiegelt config.py::_TIBIA_LIMITS (Cross-Check test_config.py) und
-       die per-Bein-Overrides in hexapod.urdf.xacro. -->
+  <!-- Stage 1 / Teil 2.1 (2026-06-02): Tibia-Beuge auf das strikt-symmetrische
+       Mechanik-Maximum +2.50 (143°) freigeschaltet (war +1.30, konservativ).
+       Einseitiges Knie: Streck -1.00 bleibt (nie genutzt). +2.50 = größter Wert,
+       den ALLE 6 Servos puls-seitig erreichen (leg_5-bound, Reserve fürs
+       pulse_zero-Peilrauschen). Spiegelt config.py::_TIBIA_LIMITS (Cross-Check
+       test_config.py) + die per-Bein-Overrides in hexapod.urdf.xacro.
+       Sicherheit pose-abhängig (Femur beim Laufen oben) per Design-Zeit-Envelope,
+       kein Laufzeit-Check (Weg B deferred). Plan: phase_13_stage_1_tibia_unlock_plan.md. -->
   <xacro:property name="tibia_lower"  value="-1.00"/>
-  <xacro:property name="tibia_upper"  value=" 1.30"/>
+  <xacro:property name="tibia_upper"  value=" 2.50"/>
   <xacro:property name="joint_effort"   value="5.0"/>  <!-- effort/velocity: vom Servo-DB -->
   <xacro:property name="joint_velocity" value="2.0"/>
