Commit message: entered new leg properties into the system

File: src/hexapod_description/urdf/hexapod.ros2_control.xacro (robot description, xacro)
@@ -78,29 +78,33 @@
          Werte sind synchron zu hexapod.urdf.xacro <xacro:leg ...>-
          Aufrufen. Plugin liest diese als <param min/max> und validiert
-         via Calibration::set_joint_limits. -->
+         via Calibration::set_joint_limits.
+         AKTUELL (Bein-Umbau leg_changes): Tibia -0.28 / +2.50 (die hier historisch
+         genannten ±1.161 sind seit dem Stage-1-Unlock ueberholt). Femur ±1.57,
+         Coxa ±0.415. Diese 6×3 Werte == hexapod.urdf.xacro, geprueft per
+         test_per_leg_limits (hexapod_kinematics). -->
     <!-- Bein 1 (front-right) -->
     <xacro:joint_iface name="leg_1_coxa_joint"  lower="-0.415" upper="0.415" initial="-0.069"/>
     <xacro:joint_iface name="leg_1_femur_joint" lower="-1.57" upper="1.57" initial="-0.469"/>
-    <xacro:joint_iface name="leg_1_tibia_joint" lower="-1.00" upper="2.50" initial="0.4946"/>
+    <xacro:joint_iface name="leg_1_tibia_joint" lower="-0.28" upper="2.50" initial="0.4946"/>
     <!-- Bein 2 (mid-right) -->
     <xacro:joint_iface name="leg_2_coxa_joint"  lower="-0.415" upper="0.415" initial="0.156"/>
     <xacro:joint_iface name="leg_2_femur_joint" lower="-1.57" upper="1.57" initial="-0.637"/>
-    <xacro:joint_iface name="leg_2_tibia_joint" lower="-1.00" upper="2.50" initial="0.5181"/>
+    <xacro:joint_iface name="leg_2_tibia_joint" lower="-0.28" upper="2.50" initial="0.5181"/>
     <!-- Bein 3 (back-right) -->
     <xacro:joint_iface name="leg_3_coxa_joint"  lower="-0.415" upper="0.415" initial="-0.111"/>
     <xacro:joint_iface name="leg_3_femur_joint" lower="-1.57" upper="1.57" initial="-0.439"/>
-    <xacro:joint_iface name="leg_3_tibia_joint" lower="-1.00" upper="2.50" initial="0.2591"/>
+    <xacro:joint_iface name="leg_3_tibia_joint" lower="-0.28" upper="2.50" initial="0.2591"/>
     <!-- Bein 4 (back-left) -->
     <xacro:joint_iface name="leg_4_coxa_joint"  lower="-0.415" upper="0.415" initial="0.026"/>
     <xacro:joint_iface name="leg_4_femur_joint" lower="-1.57" upper="1.57" initial="-0.477"/>
-    <xacro:joint_iface name="leg_4_tibia_joint" lower="-1.00" upper="2.50" initial="0.4286"/>
+    <xacro:joint_iface name="leg_4_tibia_joint" lower="-0.28" upper="2.50" initial="0.4286"/>
     <!-- Bein 5 (mid-left) -->
     <xacro:joint_iface name="leg_5_coxa_joint"  lower="-0.415" upper="0.415" initial="0.104"/>
     <xacro:joint_iface name="leg_5_femur_joint" lower="-1.57" upper="1.57" initial="-0.419"/>
-    <xacro:joint_iface name="leg_5_tibia_joint" lower="-1.00" upper="2.50" initial="0.1978"/>
+    <xacro:joint_iface name="leg_5_tibia_joint" lower="-0.28" upper="2.50" initial="0.1978"/>
     <!-- Bein 6 (front-left) -->
     <xacro:joint_iface name="leg_6_coxa_joint"  lower="-0.415" upper="0.415" initial="0.052"/>
     <xacro:joint_iface name="leg_6_femur_joint" lower="-1.57" upper="1.57" initial="-0.496"/>
-    <xacro:joint_iface name="leg_6_tibia_joint" lower="-1.00" upper="2.50" initial="0.3503"/>
+    <xacro:joint_iface name="leg_6_tibia_joint" lower="-0.28" upper="2.50" initial="0.3503"/>
   </ros2_control>
   <!--

File: src/hexapod_description/urdf/hexapod.urdf.xacro (robot description, xacro)
@@ -71,5 +71,9 @@
        oben) per Envelope-Check, kein Laufzeit-Kollisions-Check (Weg B deferred).
        Cal-Modell: docs_raspi/phase_13_stage_0_6_6_tibia_recal_plan.md.
-       Unlock-Plan: docs_raspi/phase_13_stage_1_tibia_unlock_plan.md. -->
+       Unlock-Plan: docs_raspi/phase_13_stage_1_tibia_unlock_plan.md.
+       Bein-Umbau (leg_changes, kuerzere Femur+Tibia): Streck-Limit -1.00 → -0.28
+       (neuer, viel engerer Ueberstreck-Anschlag der kurzen Tibia; handover.md §1),
+       Beuge +2.50 unveraendert. Symmetrie ueber alle 6 Beine + Sync urdf↔ros2_control
+       jetzt per test_per_leg_limits (hexapod_kinematics) abgesichert. -->
   <xacro:leg id="1"
              mount_x="${ body_length/2}" mount_y="${-body_width/2}"
@@ -77,5 +81,5 @@
              coxa_lower="-0.415"  coxa_upper="0.415"
              femur_lower="-1.57"  femur_upper="1.57"
-             tibia_lower="-1.00"  tibia_upper="2.50"/>
+             tibia_lower="-0.28"  tibia_upper="2.50"/>
   <xacro:leg id="2"
              mount_x="0"                 mount_y="${-body_width_middle/2}"
@@ -83,5 +87,5 @@
              coxa_lower="-0.415"  coxa_upper="0.415"
              femur_lower="-1.57"  femur_upper="1.57"
-             tibia_lower="-1.00"  tibia_upper="2.50"/>
+             tibia_lower="-0.28"  tibia_upper="2.50"/>
   <xacro:leg id="3"
              mount_x="${-body_length/2}" mount_y="${-body_width/2}"
@@ -89,5 +93,5 @@
              coxa_lower="-0.415"  coxa_upper="0.415"
              femur_lower="-1.57"  femur_upper="1.57"
-             tibia_lower="-1.00"  tibia_upper="2.50"/>
+             tibia_lower="-0.28"  tibia_upper="2.50"/>
   <xacro:leg id="4"
              mount_x="${-body_length/2}" mount_y="${ body_width/2}"
@@ -95,5 +99,5 @@
              coxa_lower="-0.415"  coxa_upper="0.415"
              femur_lower="-1.57"  femur_upper="1.57"
-             tibia_lower="-1.00"  tibia_upper="2.50"/>
+             tibia_lower="-0.28"  tibia_upper="2.50"/>
   <xacro:leg id="5"
              mount_x="0"                 mount_y="${ body_width_middle/2}"
@@ -101,5 +105,5 @@
              coxa_lower="-0.415"  coxa_upper="0.415"
              femur_lower="-1.57"  femur_upper="1.57"
-             tibia_lower="-1.00"  tibia_upper="2.50"/>
+             tibia_lower="-0.28"  tibia_upper="2.50"/>
   <xacro:leg id="6"
              mount_x="${ body_length/2}" mount_y="${ body_width/2}"
@@ -107,5 +111,5 @@
              coxa_lower="-0.415"  coxa_upper="0.415"
              femur_lower="-1.57"  femur_upper="1.57"
-             tibia_lower="-1.00"  tibia_upper="2.50"/>
+             tibia_lower="-0.28"  tibia_upper="2.50"/>
   <!-- ===== Gazebo-spezifische Eigenschaften (Reibung an Foot-Kugeln) ===== -->
   <xacro:include filename="hexapod.gazebo.xacro"/>

File: src/hexapod_description/urdf/hexapod_physical_properties.xacro (robot description, xacro)
@@ -11,11 +11,17 @@
   <xacro:property name="coxa_width"  value="0.0254"/>
   <xacro:property name="coxa_height" value="0.0582"/>
-  <xacro:property name="femur_length" value="0.07994"/>
+  <xacro:property name="femur_length" value="0.060"/>
   <xacro:property name="femur_width"  value="0.059"/>
   <xacro:property name="femur_height" value="0.020"/>
-  <xacro:property name="tibia_length" value="0.200"/>
+  <xacro:property name="tibia_length" value="0.134"/>
   <xacro:property name="tibia_width"  value="0.012"/>
   <xacro:property name="tibia_height" value="0.012"/>
-  <xacro:property name="segment_mass" value="0.1167"/>
+  <!-- Bein-Umbau (leg_changes): Femur+Tibia kuerzer → eigene Massen statt
+       gemeinsamem segment_mass. Coxa unveraendert (0.1167). Beide neuen Segmente
+       zusammen 220 g, Tibia +15 % (handover.md §1). Inertien propagieren via
+       inertials.xacro (Box-Formel + 1e-5-Clamp), nicht von Hand rechnen. -->
+  <xacro:property name="coxa_mass"  value="0.1167"/>
+  <xacro:property name="femur_mass" value="0.102"/>
+  <xacro:property name="tibia_mass" value="0.118"/>
   <!-- Foot (Kugel am Tibia-Ende fuer Punktkontakt, wird in Stufe B genutzt) -->
   <xacro:property name="foot_radius" value="0.008"/>
@@ -26,13 +32,14 @@
   <xacro:property name="femur_lower"  value="-1.57"/>
   <xacro:property name="femur_upper"  value=" 1.57"/>
-  <!-- Stage 1 / Teil 2.1 (2026-06-02): Tibia-Beuge auf das strikt-symmetrische
-       Mechanik-Maximum +2.50 (143°) freigeschaltet (war +1.30, konservativ).
-       Einseitiges Knie: Streck -1.00 bleibt (nie genutzt). +2.50 = größter Wert,
-       den ALLE 6 Servos puls-seitig erreichen (leg_5-bound, Reserve fürs
-       pulse_zero-Peilrauschen). Spiegelt config.py::_TIBIA_LIMITS (Cross-Check
-       test_config.py) + die per-Bein-Overrides in hexapod.urdf.xacro.
-       Sicherheit pose-abhängig (Femur beim Laufen oben) per Design-Zeit-Envelope,
-       kein Laufzeit-Check (Weg B deferred). Plan: phase_13_stage_1_tibia_unlock_plan.md. -->
-  <xacro:property name="tibia_lower"  value="-1.00"/>
+  <!-- Tibia-Beuge +2.50 (143°) = strikt-symmetrisches Mechanik-Maximum, das ALLE
+       6 Servos puls-seitig erreichen (leg_5-bound). Streck-Anschlag durch den
+       Bein-Umbau (leg_changes, kuerzere Tibia) von -1.00 auf -0.28 verengt — der
+       neue, viel engere Ueberstreck-Anschlag der kurzen Tibia (handover.md §1).
+       Property = Default/Referenz; maßgeblich sind die per-Bein-Werte in
+       hexapod.urdf.xacro + hexapod.ros2_control.xacro. Symmetrie ueber alle 6
+       Beine + Sync der beiden URDF-Quellen via test_per_leg_limits, config.py-
+       Mirror via test_config.py. Sicherheit pose-abhaengig per Design-Zeit-
+       Envelope, kein Laufzeit-Check. -->
+  <xacro:property name="tibia_lower"  value="-0.28"/>
   <xacro:property name="tibia_upper"  value=" 2.50"/>
   <xacro:property name="joint_effort"   value="5.0"/>  <!-- effort/velocity: vom Servo-DB -->

File: src/hexapod_description/urdf/leg.xacro (robot description, xacro)
@@ -42,5 +42,5 @@
         </geometry>
       </collision>
-      <xacro:box_inertia mass="${segment_mass}"
+      <xacro:box_inertia mass="${coxa_mass}"
                          x="${coxa_length}" y="${coxa_width}" z="${coxa_height}"/>
     </link>
@@ -68,5 +68,5 @@
         </geometry>
       </collision>
-      <xacro:box_inertia mass="${segment_mass}"
+      <xacro:box_inertia mass="${femur_mass}"
                          x="${femur_length}" y="${femur_width}" z="${femur_height}"/>
     </link>
@@ -94,5 +94,5 @@
         </geometry>
       </collision>
-      <xacro:box_inertia mass="${segment_mass}"
+      <xacro:box_inertia mass="${tibia_mass}"
                          x="${tibia_length}" y="${tibia_width}" z="${tibia_height}"/>
     </link>

Commit message: stage 3 envelope done, stage 4 prepared

File: src/hexapod_description/urdf/hexapod.ros2_control.xacro (robot description, xacro)
@@ -85,26 +85,26 @@
     <!-- Bein 1 (front-right) -->
     <xacro:joint_iface name="leg_1_coxa_joint"  lower="-0.415" upper="0.415" initial="-0.069"/>
-    <xacro:joint_iface name="leg_1_femur_joint" lower="-1.57" upper="1.57" initial="-0.469"/>
-    <xacro:joint_iface name="leg_1_tibia_joint" lower="-0.28" upper="2.50" initial="0.4946"/>
+    <xacro:joint_iface name="leg_1_femur_joint" lower="-1.57" upper="1.57" initial="-0.7732"/>
+    <xacro:joint_iface name="leg_1_tibia_joint" lower="-0.28" upper="2.50" initial="0.8491"/>
     <!-- Bein 2 (mid-right) -->
     <xacro:joint_iface name="leg_2_coxa_joint"  lower="-0.415" upper="0.415" initial="0.156"/>
-    <xacro:joint_iface name="leg_2_femur_joint" lower="-1.57" upper="1.57" initial="-0.637"/>
-    <xacro:joint_iface name="leg_2_tibia_joint" lower="-0.28" upper="2.50" initial="0.5181"/>
+    <xacro:joint_iface name="leg_2_femur_joint" lower="-1.57" upper="1.57" initial="-0.9523"/>
+    <xacro:joint_iface name="leg_2_tibia_joint" lower="-0.28" upper="2.50" initial="0.9089"/>
     <!-- Bein 3 (back-right) -->
     <xacro:joint_iface name="leg_3_coxa_joint"  lower="-0.415" upper="0.415" initial="-0.111"/>
-    <xacro:joint_iface name="leg_3_femur_joint" lower="-1.57" upper="1.57" initial="-0.439"/>
-    <xacro:joint_iface name="leg_3_tibia_joint" lower="-0.28" upper="2.50" initial="0.2591"/>
+    <xacro:joint_iface name="leg_3_femur_joint" lower="-1.57" upper="1.57" initial="-0.8431"/>
+    <xacro:joint_iface name="leg_3_tibia_joint" lower="-0.28" upper="2.50" initial="1.0046"/>
     <!-- Bein 4 (back-left) -->
     <xacro:joint_iface name="leg_4_coxa_joint"  lower="-0.415" upper="0.415" initial="0.026"/>
-    <xacro:joint_iface name="leg_4_femur_joint" lower="-1.57" upper="1.57" initial="-0.477"/>
-    <xacro:joint_iface name="leg_4_tibia_joint" lower="-0.28" upper="2.50" initial="0.4286"/>
+    <xacro:joint_iface name="leg_4_femur_joint" lower="-1.57" upper="1.57" initial="-0.8157"/>
+    <xacro:joint_iface name="leg_4_tibia_joint" lower="-0.28" upper="2.50" initial="1.0485"/>
     <!-- Bein 5 (mid-left) -->
     <xacro:joint_iface name="leg_5_coxa_joint"  lower="-0.415" upper="0.415" initial="0.104"/>
-    <xacro:joint_iface name="leg_5_femur_joint" lower="-1.57" upper="1.57" initial="-0.419"/>
-    <xacro:joint_iface name="leg_5_tibia_joint" lower="-0.28" upper="2.50" initial="0.1978"/>
+    <xacro:joint_iface name="leg_5_femur_joint" lower="-1.57" upper="1.57" initial="-0.8276"/>
+    <xacro:joint_iface name="leg_5_tibia_joint" lower="-0.28" upper="2.50" initial="0.9745"/>
     <!-- Bein 6 (front-left) -->
     <xacro:joint_iface name="leg_6_coxa_joint"  lower="-0.415" upper="0.415" initial="0.052"/>
-    <xacro:joint_iface name="leg_6_femur_joint" lower="-1.57" upper="1.57" initial="-0.496"/>
-    <xacro:joint_iface name="leg_6_tibia_joint" lower="-0.28" upper="2.50" initial="0.3503"/>
+    <xacro:joint_iface name="leg_6_femur_joint" lower="-1.57" upper="1.57" initial="-0.7697"/>
+    <xacro:joint_iface name="leg_6_tibia_joint" lower="-0.28" upper="2.50" initial="0.8464"/>
   </ros2_control>
   <!--

File: src/hexapod_description/urdf/hexapod_physical_properties.xacro (robot description, xacro)
@@ -28,6 +28,9 @@
   <xacro:property name="foot_mass"   value="0.005"/>
   <!-- Joint-Limits (physisch verifiziert, siehe 00_conventions.md §11.4) -->
-  <xacro:property name="coxa_lower"   value="-1.57"/>
-  <xacro:property name="coxa_upper"   value=" 1.57"/>
+  <!-- Coxa: ±0.415 = echte mech. Grenze (rad+PWM doppelt verifiziert); die
+       frueheren ±1.57 waren die Datenblatt-Verifikations-Cal. Property +
+       config.py jetzt konsistent zu den per-Bein-URDF-Werten (leg_changes S3). -->
+  <xacro:property name="coxa_lower"   value="-0.415"/>
+  <xacro:property name="coxa_upper"   value=" 0.415"/>
   <xacro:property name="femur_lower"  value="-1.57"/>
   <xacro:property name="femur_upper"  value=" 1.57"/>
