Commit message: added imu general functionality to gazebo and rviz, not real use for now

File: src/hexapod_description/urdf/hexapod.urdf.xacro (robot description, xacro)
@@ -6,4 +6,8 @@
        gestartet (siehe hexapod_bringup/launch/sim.launch.py). -->
   <xacro:arg name="enable_foot_contact" default="true"/>
+  <!-- Block A5 Stufe 0: Toggle für IMU (BNO-055). Default true; bei false kein
+       imu_link/Sensor, Bridge + imu_monitor starten im Launch nicht. Der
+       gz-IMU-Sensor-Block ist zusätzlich use_sim-geguarded (nur Sim). -->
+  <xacro:arg name="enable_imu" default="true"/>
   <!-- Phase 9 Stufe F: Sim/HW-Switch + Hardware-Parameter.
        Diese drei Args sind die "öffentliche Schnittstelle" des URDF-
@@ -76,4 +80,6 @@
        Beuge +2.50 unveraendert. Symmetrie ueber alle 6 Beine + Sync urdf↔ros2_control
        jetzt per test_per_leg_limits (hexapod_kinematics) abgesichert. -->
+  <!-- leg_1-Femur GRÜN als Orientierungs-Marker (vorne rechts) — sichtbar in
+       Gazebo + RViz, macht Front/Bein-Zuordnung beim Balance-/Kipp-Test eindeutig. -->
   <xacro:leg id="1"
              mount_x="${ body_length/2}" mount_y="${-body_width/2}"
@@ -81,5 +87,6 @@
              coxa_lower="-0.415"  coxa_upper="0.415"
              femur_lower="-1.57"  femur_upper="1.57"
-             tibia_lower="-0.28"  tibia_upper="2.50"/>
+             tibia_lower="-0.28"  tibia_upper="2.50"
+             femur_material="green"/>
   <xacro:leg id="2"
              mount_x="0"                 mount_y="${-body_width_middle/2}"
@@ -120,3 +127,7 @@
     <xacro:include filename="hexapod.foot_contact.xacro"/>
   </xacro:if>
+  <!-- ===== IMU (Block A5 Stufe 0, conditional) ===== -->
+  <xacro:if value="$(arg enable_imu)">
+    <xacro:include filename="hexapod.imu.xacro"/>
+  </xacro:if>
 </robot>

File: src/hexapod_description/urdf/leg.xacro (robot description, xacro)
@@ -17,5 +17,6 @@
                                   femur_upper:=^|${femur_upper}|
                                   tibia_lower:=^|${tibia_lower}|
-                                  tibia_upper:=^|${tibia_upper}|">
+                                  tibia_upper:=^|${tibia_upper}|
+                                  femur_material:=orange">
     <!-- ===== Coxa ===== -->
     <joint name="leg_${id}_coxa_joint" type="revolute">
@@ -60,5 +61,5 @@
           <box size="${femur_length} ${femur_width} ${femur_height}"/>
         </geometry>
-        <material name="orange"/>
+        <material name="${femur_material}"/>
       </visual>
       <collision>

File: src/hexapod_description/urdf/materials.xacro (robot description, xacro)
@@ -4,3 +4,4 @@
   <material name="grey">  <color rgba="0.4 0.4 0.4 1.0"/></material>
   <material name="black"> <color rgba="0.1 0.1 0.1 1.0"/></material>
+  <material name="green"> <color rgba="0.1 0.8 0.1 1.0"/></material>
 </robot>
